File: libre-debugger.sch (KiCad schematic (older format))
At the start: 82 parts, among them J1 USB_C_Receptacle_USB2.0, J2 Conn_ST_STDC14, J4 Conn_01x16, Q1 2N7002, SW1 SW_SPDT, SW2 SW_Push, U1 FT2232H, U10 74LVC1G125, U11 74LVC1G125, U12 74LVC1G125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

Commit message: Replace LDO: MIC5504 -> XC6026
Available on JLCPCB as Basic Part.
Many alternative MPNs available for this new footprint, so not an issue.
Parts:
- removed U2: MIC5504-3.3YM5, Package_TO_SOT_SMD:SOT-23-5, symbol Regulator_Linear:MIC5504-3.3YM5
- added U2: XC6206PxxxMR, Package_TO_SOT_SMD:SOT-23, symbol Regulator_Linear:XC6206PxxxMR
Connections:
- wire segments 371 -> 368
Changed lines of the file:
@@
 	1    0    0    -1
 $EndComp
-Wire Wire Line
-	2750 3100 2900 3100
-Connection ~ 2750 3100
-Wire Wire Line
-	2650 3100 2750 3100
 Connection ~ 2650 3100
 Wire Wire Line
@@
 Wire Wire Line
 	3900 3100 4150 3100
-Wire Wire Line
-	3300 3600 3300 3500
 $Comp
 L power:GND #PWR010
@@
 	0    1    1    0
 $EndComp
-$Comp
-L Regulator_Linear:MIC5504-3.3YM5 U2
-U 1 1 5C788716
-P 3300 3200
-F 0 "U2" H 3300 3567 50  0000 C CNN
-F 1 "MIC5504-3.3YM5" H 3300 3476 50  0000 C CNN
-F 2 "Package_TO_SOT_SMD:SOT-23-5" H 3300 2800 50  0001 C CNN
-F 3 "http://ww1.microchip.com/downloads/en/DeviceDoc/MIC550X.pdf" H 3050 3450 50  0001 C CNN
-F 4 "C88419" H 3300 3200 50  0001 C CNN "LCSC_PN"
-F 5 "MIC5504-3.3YM5-TR" H 3300 3200 50  0001 C CNN "MPN"
-F 6 "Microchip" H 3300 3200 50  0001 C CNN "Manufacturer"
-	1    3300 3200
-	1    0    0    -1
-$EndComp
-Wire Wire Line
-	2900 3300 2750 3300
-Wire Wire Line
-	2750 3100 2750 3300
 Wire Wire Line
 	11700 2350 11700 2300
@@
 Connection ~ 4150 3100
 Wire Wire Line
-	3900 3100 3700 3100
-Wire Wire Line
 	4150 3100 4650 3100
 Wire Wire Line
@@
 Wire Wire Line
 	8400 9200 8400 9350
+Wire Wire Line
+	3300 3400 3300 3600
+Wire Wire Line
+	2650 3100 3000 3100
+Wire Wire Line
+	3600 3100 3900 3100
+$Comp
+L Regulator_Linear:XC6206PxxxMR U2
+U 1 1 5DBFF3BB
+P 3300 3100
+F 0 "U2" H 3300 3342 50  0000 C CNN
+F 1 "XC6206PxxxMR" H 3300 3251 50  0000 C CNN
+F 2 "Package_TO_SOT_SMD:SOT-23" H 3300 3325 50  0001 C CIN
+F 3 "https://www.torexsemi.com/file/xc6206/XC6206.pdf" H 3300 3100 50  0001 C CNN
+F 4 "C5446" H 3300 3100 50  0001 C CNN "LCSC_PN"
+F 5 "XC6206P332MR" H 3300 3100 50  0001 C CNN "MPN"
+F 6 "Torex Semiconductor" H 3300 3100 50  0001 C CNN "Manufacturer"
+	1    3300 3100
+	1    0    0    -1
+$EndComp
 $EndSCHEMATC

Commit message: Use 4u7 caps for LDO input and output too
Minimum size recommended is 1uF input and 1uF output.
But given capacitance derating vs DC voltage, it is probably
a good idea to go for a higher value. That reduces the number
of MPNs too.
Parts:
- C1, C2: value 1u -> 4u7; LCSC_PN (none) -> C19666; MPN (none) -> CL10A475KO8NNNC; Manufacturer (none) -> Samsung Electro-Mechanics
Other:
- note removed: "maybe 4u7 in n out?"
Changed lines of the file:
@@
 Wire Wire Line
 	5300 5550 5250 5550
-Text Notes 2900 2800 0    50   ~ 10
-maybe 4u7 in n out?
 Wire Wire Line
 	2550 3100 2650 3100
@@
 P 2550 3400
 F 0 "C1" H 2665 3446 50  0000 L CNN
-F 1 "1u" H 2665 3355 50  0000 L CNN
+F 1 "4u7" H 2665 3355 50  0000 L CNN
 F 2 "Capacitor_SMD:C_0603_1608Metric" H 2588 3250 50  0001 C CNN
 F 3 "~" H 2550 3400 50  0001 C CNN
+F 4 "C19666" H 2550 3400 50  0001 C CNN "LCSC_PN"
+F 5 "CL10A475KO8NNNC" H 2550 3400 50  0001 C CNN "MPN"
+F 6 "Samsung Electro-Mechanics" H 2550 3400 50  0001 C CNN "Manufacturer"
 	1    2550 3400
 	1    0    0    -1
@@
 P 3900 3400
 F 0 "C2" H 4015 3446 50  0000 L CNN
-F 1 "1u" H 4015 3355 50  0000 L CNN
+F 1 "4u7" H 4015 3355 50  0000 L CNN
 F 2 "Capacitor_SMD:C_0603_1608Metric" H 3938 3250 50  0001 C CNN
 F 3 "~" H 3900 3400 50  0001 C CNN
+F 4 "C19666" H 3900 3400 50  0001 C CNN "LCSC_PN"
+F 5 "CL10A475KO8NNNC" H 3900 3400 50  0001 C CNN "MPN"
+F 6 "Samsung Electro-Mechanics" H 3900 3400 50  0001 C CNN "Manufacturer"
 	1    3900 3400
 	1    0    0    -1

Commit message: Add many MPNs including alternatives
Parts:
- C1, C17, C2, C5, C6, C7: MPN CL10A475KO8NNNC -> (none); MPN2 (none) -> CL10A475KO8NNNC; Manufacturer Samsung Electro-Mechanics -> (none); Manufacturer2 (none) -> Samsung Electro-Mechanics
- C10, C11, C12, C13, C14, C15, C16, C18, C19, C20, C21, C22, C8, C9: MPN CC0603KRX7R9BB104 -> (none); MPN2 (none) -> CC0603KRX7R9BB104; Manufacturer Yageo -> (none); Manufacturer2 (none) -> Yageo
- C3, C4: MPN CL10C270JB8NNNC -> C0603C270J5GAC; MPN2 (none) -> CL10C270JB8NNNC; Manufacturer Samsung Electro-Mechanics -> Kemet; Manufacturer2 (none) -> Samsung Electro-Mechanics
- D1, D2, D3, D4, D5, D6: MPN 19-217/GHC-YR1S2/3T -> (none); MPN2 (none) -> 19-217/GHC-YR1S2/3T; Manufacturer Everlight Elec -> (none); Manufacturer2 (none) -> Everlight Elec
- J1: MPN (none) -> USB4085-GF-A; Manufacturer (none) -> GCT
- J2: MPN (none) -> FTSH-107-01-F-DV-K; Manufacturer (none) -> Samtec
- J4: MPN (none) -> M20-9991645; MPN2 (none) -> 2057-PH1-16-UA-ND; Manufacturer (none) -> Harwin; Manufacturer2 (none) -> Adam Tech
- Q1: MPN (none) -> 2N7002-7-F; MPN2 (none) -> 2N7002; Manufacturer (none) -> Diodes Incorporated; Manufacturer2 (none) -> Changjiang Electronics Tech (CJ)
- SW1: MPN (none) -> EG1215AA; MPN2 (none) -> SSSS811101; Manufacturer (none) -> E-Switch; Manufacturer2 (none) -> Alps
- U10, U11, U12, U5, U7, U8, U9: MPN2 (none) -> SN74LVC1G125DCK; Manufacturer2 (none) -> Texas Instruments
- U2: MPN2 (none) -> AP2120N-3.3TRG1; Manufacturer2 (none) -> Diodes Incorporated
- U3: MPN (none) -> SRV05-4HTG-D; MPN2 (none) -> SRV05-4-P-T7; Manufacturer (none) -> Littelfuse; Manufacturer2 (none) -> ProTek Devices
- U6: MPN2 (none) -> SN74LVC1G126DCK; Manufacturer2 (none) -> Texas Instruments
- Y1: MPN X322512MSB4SI -> ABM8-12.000MHZ-20-B1U-T; MPN2 (none) -> X322512MSB4SI; Manufacturer Yangxing Tech -> Abracon LLC; Manufacturer2 (none) -> Yangxing Tech; Tolerance (none) -> 10PPM
